Commit message: urdf working

File: test_urdf.urdf (robot description, URDF)
Before this commit: robot test_robot, 6 links, 5 joints
Links:
- link base_link: mass None -> 1572.9; geometry collision cylinder length=0.056 radius=0.1; visual cylinder length=0.056 radius=0.1
- link link_1: mass None -> 1385.5; geometry collision cylinder length=0.0386 radius=0.03; visual cylinder length=0.0386 radius=0.03
- link link_2: mass None -> 958.62; geometry collision cylinder length=0.12 radius=0.03; visual cylinder length=0.12 radius=0.03
- link link_3: mass None -> 710.03; geometry collision cylinder length=0.09 radius=0.03; visual cylinder length=0.09 radius=0.03
- link link_4: mass None -> 173.73; geometry collision cylinder length=0.028/ radius=0.03; visual cylinder length=0.028/ radius=0.03
- link link_5: mass None -> 72.17; geometry collision cylinder length=0.08 radius=0.03; visual cylinder length=0.08 radius=0.03

Commit message: bug

File: test_urdf.urdf (robot description, URDF)
Before this commit: robot test_robot, 6 links, 5 joints
Links:
- link link_4: geometry collision cylinder length=0.028 radius=0.03; visual cylinder length=0.028 radius=0.03
