Commit message: changes

File: bb_test.urdf (robot description, URDF)
Before this commit: robot kuka_kr210, 1 links, 0 joints
Links:
- link base_link: geometry collision mesh filename=visuals/stl/Base.stl; visual mesh filename=visuals/meshes/Base.dae

Commit message: changes

File: bb_test.urdf (robot description, URDF)
Before this commit: robot kuka_kr210, 1 links, 0 joints
Links:
- added link arm_link_1, mass 1385.5; collision mesh filename=visuals/stl/Arm_01.stl; visual mesh filename=visuals/meshes/Arm_01.dae
- added link arm_link_2, mass 1385.5; collision mesh filename=visuals/stl/Arm_02_v3.stl; visual mesh filename=visuals/meshes/Arm_02_v3.dae
- added link waist_link, mass 1385.5; collision mesh filename=visuals/stl/waist.stl; visual mesh filename=visuals/meshes/waist.dae
- added link wrist_link_1, mass 1385.5; collision mesh filename=visuals/stl/Arm_03.stl; visual mesh filename=visuals/meshes/Arm_03.dae
Joints:
- added joint joint_a1: type revolute, parent base_link, child waist_link, origin xyz=-0.00262 0.00097586 0.33099 rpy=0 0 0, axis 0 0 1, limit lower=-3.228859205 upper=3.228859205 effort=0 velocity=2.146755039
- added joint joint_a2: type revolute, parent waist_link, child arm_link_1, origin xyz=0.35277 -0.037476 0.4192 rpy=0 0 0, axis 0 1 0, limit lower=-0.785398185 upper=1.483529905 effort=0 velocity=2.007128695
- added joint joint_a3: type revolute, parent arm_link_1, child arm_link_2, origin xyz=-9.8483E-05 -0.1475 1.2499 rpy=0 0 0, axis 0 1 0, limit lower=-3.66519153 upper=1.134464045 effort=0 velocity=1.954768816
- added joint joint_a4: type revolute, parent arm_link_2, child wrist_link_1, origin xyz=0.95795 0.184 -0.055059 rpy=0 0 0, axis 1 0 0, limit lower=-6.10865255 upper=6.10865255 effort=0 velocity=3.124139447

Commit message: changes

File: bb_test.urdf (robot description, URDF)
Before this commit: robot kuka_kr210, 5 links, 4 joints
Links:
- added link wrist_link_2, mass 1385.5; collision mesh filename=visuals/stl/Gripper_base.stl; visual mesh filename=visuals/meshes/Gripper_base.dae
Joints:
- added joint joint_a5: type revolute, parent wrist_link_1, child wrist_link_2, origin xyz=0.542 0 0 rpy=0 0 0, axis 0 1 0, limit lower=-2.181661625 upper=2.181661625 effort=0 velocity=3.001966396

Commit message: last call

File: bb_test.urdf (robot description, URDF)
Before this commit: robot kuka_kr210, 6 links, 5 joints
Links:
- added link endpoint_link, mass 1385.5; collision cylinder length=0.6 radius=0.01; visual cylinder length=0.6 radius=0.01
- link arm_link_1: geometry collision mesh filename=visuals/meshes/Arm_01.dae; visual mesh filename=visuals/meshes/Arm_01.dae
- link arm_link_2: geometry collision mesh filename=visuals/meshes/Arm_02_v3.dae; visual mesh filename=visuals/meshes/Arm_02_v3.dae
- link waist_link: geometry collision mesh filename=visuals/meshes/Waist.dae; visual mesh filename=visuals/meshes/Waist.dae
- link wrist_link_1: geometry collision mesh filename=visuals/meshes/Arm_03.dae; visual mesh filename=visuals/meshes/Arm_03.dae
- link wrist_link_2: geometry collision mesh filename=visuals/meshes/Gripper_base.dae; visual mesh filename=visuals/meshes/Gripper_base.dae
Joints:
- removed joint joint_a1
- removed joint joint_a2
- removed joint joint_a3
- removed joint joint_a4
- removed joint joint_a5
- added joint elbow_joint: type revolute, parent arm_link_1, child arm_link_2, origin xyz=0 0.25 1.3 rpy=0 0 3.14, axis 1 0 0, limit lower=-0.786 upper=0.786 effort=100 velocity=1.954768816
- added joint joint_a6: type revolute, parent wrist_link_2, child endpoint_link, origin xyz=-0.175 -0.25 1.06 rpy=0 0 0, axis -1 0 0, limit lower=-2.181661625 upper=2.181661625 effort=100 velocity=3.001966396
- added joint shoulder_joint: type revolute, parent waist_link, child arm_link_1, origin xyz=0 -0.15 0.24 rpy=0 0 0, axis 1 0 0, limit lower=-1.179 upper=1.5327 effort=100 velocity=2.007128695
- added joint waist_joint: type revolute, parent base_link, child waist_link, origin xyz=0 0 0.56 rpy=0 0 0, axis 0 0 -1, limit lower=-1.082 upper=1.082 effort=100 velocity=2.146755039
- added joint wrist_extention_joint: type revolute, parent wrist_link_1, child wrist_link_2, origin xyz=0 0.25 0 rpy=0 0 0, axis -1 0 0, limit lower=-1.122 upper=0.9537 effort=100 velocity=3.001966396
- added joint wrist_roll_joint: type revolute, parent arm_link_2, child wrist_link_1, origin xyz=0 0.035 1.18 rpy=0 0 0, axis 0 0 1, limit lower=-2.244 upper=1.4025 effort=100 velocity=3.124139447
